File: kicad_files/audioamp.sch (KiCad schematic (older format))
At the start: 27 parts, among them J1 Conn_01x03_Female, J2 Conn_01x02_Female, U1 TDA2030, U2 TDA2030

Commit message: Adicionados comentários e PDF gerado
Other:
- note added: "Amplificador e saída"
- note added: "Conectores"
- note added: "Filtro passa-baixas"
- moved on the sheet: C1, C2, C3, C4, C5, C6, C7, C8, C9, D1, D2, D3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

Commit message: Adicionados footprints aos componentes
Parts:
- C1, C2, C3, C5, C6, C9: footprint (none) -> Capacitor_THT:CP_Radial_D5.0mm_P2.50mm
- C4, C7, C8: footprint (none) -> Capacitor_THT:C_Disc_D4.7mm_W2.5mm_P5.00mm
- J1: footprint (none) -> TerminalBlock:TerminalBlock_bornier-3_P5.08mm
- J2, LS1: footprint (none) -> TerminalBlock:TerminalBlock_bornier-2_P5.08mm
- R1, R2, R3, R6, R7, R8, R9: footprint (none) -> Resistor_THT:R_Axial_DIN0207_L6.3mm_D2.5mm_P7.62mm_Horizontal
- R4: footprint (none) -> Resistor_THT:R_Axial_DIN0414_L11.9mm_D4.5mm_P15.24mm_Horizontal
- R5: footprint (none) -> Resistor_THT:R_Axial_DIN0309_L9.0mm_D3.2mm_P12.70mm_Horizontal
Changed lines of the file:
@@
 F 0 "C3" H 6518 4446 50  0000 L CNN
 F 1 "100uF" H 6518 4355 50  0000 L CNN
-F 2 "" H 6438 4250 50  0001 C CNN
+F 2 "Capacitor_THT:CP_Radial_D5.0mm_P2.50mm" H 6438 4250 50  0001 C CNN
 F 3 "~" H 6400 4400 50  0001 C CNN
 	1    6400 4400
@@
 F 0 "C1" V 5705 2750 50  0000 C CNN
 F 1 "1uF" V 5614 2750 50  0000 C CNN
-F 2 "" H 5488 2600 50  0001 C CNN
+F 2 "Capacitor_THT:CP_Radial_D5.0mm_P2.50mm" H 5488 2600 50  0001 C CNN
 F 3 "~" H 5450 2750 50  0001 C CNN
 	1    5450 2750
@@
 F 0 "C2" H 5968 3746 50  0000 L CNN
 F 1 "22uF" H 5968 3655 50  0000 L CNN
-F 2 "" H 5888 3550 50  0001 C CNN
+F 2 "Capacitor_THT:CP_Radial_D5.0mm_P2.50mm" H 5888 3550 50  0001 C CNN
 F 3 "~" H 5850 3700 50  0001 C CNN
 	1    5850 3700
@@
 F 0 "C9" H 8668 3846 50  0000 L CNN
 F 1 "22uF" H 8668 3755 50  0000 L CNN
-F 2 "" H 8588 3650 50  0001 C CNN
+F 2 "Capacitor_THT:CP_Radial_D5.0mm_P2.50mm" H 8588 3650 50  0001 C CNN
 F 3 "~" H 8550 3800 50  0001 C CNN
 	1    8550 3800
@@
 F 0 "C6" H 7418 1696 50  0000 L CNN
 F 1 "100uF" H 7418 1605 50  0000 L CNN
-F 2 "" H 7338 1500 50  0001 C CNN
+F 2 "Capacitor_THT:CP_Radial_D5.0mm_P2.50mm" H 7338 1500 50  0001 C CNN
 F 3 "~" H 7300 1650 50  0001 C CNN
 	1    7300 1650
@@
 F 0 "C5" H 6650 4300 50  0000 L CNN
 F 1 "0.22uF" H 6550 4200 50  0000 L CNN
-F 2 "" H 6938 4050 50  0001 C CNN
+F 2 "Capacitor_THT:CP_Radial_D5.0mm_P2.50mm" H 6938 4050 50  0001 C CNN
 F 3 "~" H 6900 4200 50  0001 C CNN
 	1    6900 4200
@@
 F 0 "C4" H 6600 1650 50  0000 L CNN
 F 1 "100nF" H 6600 1550 50  0000 L CNN
-F 2 "" H 6938 1500 50  0001 C CNN
+F 2 "Capacitor_THT:C_Disc_D4.7mm_W2.5mm_P5.00mm" H 6938 1500 50  0001 C CNN
 F 3 "~" H 6900 1650 50  0001 C CNN
 	1    6900 1650
@@
 F 0 "C7" H 7000 3350 50  0000 L CNN
 F 1 "220nF" H 6950 3150 50  0000 L CNN
-F 2 "" H 7138 3100 50  0001 C CNN
+F 2 "Capacitor_THT:C_Disc_D4.7mm_W2.5mm_P5.00mm" H 7138 3100 50  0001 C CNN
 F 3 "~" H 7100 3250 50  0001 C CNN
 	1    7100 3250
@@
 F 0 "C8" H 7700 4400 50  0000 L CNN
 F 1 "100nF" H 7700 4300 50  0000 L CNN
-F 2 "" H 7988 4250 50  0001 C CNN
+F 2 "Capacitor_THT:C_Disc_D4.7mm_W2.5mm_P5.00mm" H 7988 4250 50  0001 C CNN
 F 3 "~" H 7950 4400 50  0001 C CNN
 	1    7950 4400
@@
 F 0 "R1" H 5450 3100 50  0000 L CNN
 F 1 "22K" H 5450 3000 50  0000 L CNN
-F 2 "" V 5580 3050 50  0001 C CNN
+F 2 "Resistor_THT:R_Axial_DIN0207_L6.3mm_D2.5mm_P7.62mm_Horizontal" V 5580 3050 50  0001 C CNN
 F 3 "~" H 5650 3050 50  0001 C CNN
 	1    5650 3050
@@
 F 0 "R3" V 6293 3450 50  0000 C CNN
 F 1 "22K" V 6384 3450 50  0000 C CNN
-F 2 "" V 6430 3450 50  0001 C CNN
+F 2 "Resistor_THT:R_Axial_DIN0207_L6.3mm_D2.5mm_P7.62mm_Horizontal" V 6430 3450 50  0001 C CNN
 F 3 "~" H 6500 3450 50  0001 C CNN
 	1    6500 3450
@@
 F 0 "R2" H 5920 4046 50  0000 L CNN
 F 1 "680R" H 5920 3955 50  0000 L CNN
-F 2 "" V 5780 4000 50  0001 C CNN
+F 2 "Resistor_THT:R_Axial_DIN0207_L6.3mm_D2.5mm_P7.62mm_Horizontal" V 5780 4000 50  0001 C CNN
 F 3 "~" H 5850 4000 50  0001 C CNN
 	1    5850 4000
@@
 F 0 "R9" H 8820 3096 50  0000 L CNN
 F 1 "22K" H 8820 3005 50  0000 L CNN
-F 2 "" V 8680 3050 50  0001 C CNN
+F 2 "Resistor_THT:R_Axial_DIN0207_L6.3mm_D2.5mm_P7.62mm_Horizontal" V 8680 3050 50  0001 C CNN
 F 3 "~" H 8750 3050 50  0001 C CNN
 	1    8750 3050
@@
 F 0 "R8" H 8620 4446 50  0000 L CNN
 F 1 "680R" H 8620 4355 50  0000 L CNN
-F 2 "" V 8480 4400 50  0001 C CNN
+F 2 "Resistor_THT:R_Axial_DIN0207_L6.3mm_D2.5mm_P7.62mm_Horizontal" V 8480 4400 50  0001 C CNN
 F 3 "~" H 8550 4400 50  0001 C CNN
 	1    8550 4400
@@
 F 0 "R7" V 7900 4050 50  0000 C CNN
 F 1 "22K" V 7684 4050 50  0000 C CNN
-F 2 "" V 7730 4050 50  0001 C CNN
+F 2 "Resistor_THT:R_Axial_DIN0207_L6.3mm_D2.5mm_P7.62mm_Horizontal" V 7730 4050 50  0001 C CNN
 F 3 "~" H 7800 4050 50  0001 C CNN
 	1    7800 4050
@@
 F 0 "R6" V 8007 3450 50  0000 C CNN
 F 1 "22K" V 7916 3450 50  0000 C CNN
-F 2 "" V 7730 3450 50  0001 C CNN
+F 2 "Resistor_THT:R_Axial_DIN0207_L6.3mm_D2.5mm_P7.62mm_Horizontal" V 7730 3450 50  0001 C CNN
 F 3 "~" H 7800 3450 50  0001 C CNN
 	1    7800 3450
@@
 F 0 "R4" H 6970 4546 50  0000 L CNN
 F 1 "1R" H 6970 4455 50  0000 L CNN
-F 2 "" V 6830 4500 50  0001 C CNN
+F 2 "Resistor_THT:R_Axial_DIN0414_L11.9mm_D4.5mm_P15.24mm_Horizontal" V 6830 4500 50  0001 C CNN
 F 3 "~" H 6900 4500 50  0001 C CNN
 	1    6900 4500
@@
 F 0 "J1" H 3650 1600 50  0000 C CNN
 F 1 "Conn_01x03_Female" H 3700 1750 50  0000 C CNN
-F 2 "" H 3450 1550 50  0001 C CNN
+F 2 "TerminalBlock:TerminalBlock_bornier-3_P5.08mm" H 3450 1550 50  0001 C CNN
 F 3 "~" H 3450 1550 50  0001 C CNN
 	1    3450 1550
@@
 F 0 "R5" H 7170 3596 50  0000 L CNN
 F 1 "1R" H 7170 3505 50  0000 L CNN
-F 2 "" V 7030 3550 50  0001 C CNN
+F 2 "Resistor_THT:R_Axial_DIN0309_L9.0mm_D3.2mm_P12.70mm_Horizontal" V 7030 3550 50  0001 C CNN
 F 3 "~" H 7100 3550 50  0001 C CNN
 	1    7100 3550
@@
 F 0 "J2" H 1842 1275 50  0000 C CNN
 F 1 "Conn_01x02_Female" H 1842 1366 50  0000 C CNN
-F 2 "" H 1950 1600 50  0001 C CNN
+F 2 "TerminalBlock:TerminalBlock_bornier-2_P5.08mm" H 1950 1600 50  0001 C CNN
 F 3 "~" H 1950 1600 50  0001 C CNN
 	1    1950 1600
@@
 F 0 "LS1" V 7350 2600 50  0000 R CNN
 F 1 "Speaker" V 7250 2650 50  0000 R CNN
-F 2 "" H 7050 2350 50  0001 C CNN
+F 2 "TerminalBlock:TerminalBlock_bornier-2_P5.08mm" H 7050 2350 50  0001 C CNN
 F 3 "~" H 7040 2500 50  0001 C CNN
 	1    7050 2550
@@
 $EndSheet
 $Comp
-L power:+VDC #PWR?
+L power:+VDC #PWR06
 U 1 1 5F140543
 P 2750 2600
-F 0 "#PWR?" H 2750 2500 50  0001 C CNN
+F 0 "#PWR06" H 2750 2500 50  0001 C CNN
 F 1 "+VDC" H 2750 2875 50  0000 C CNN
 F 2 "" H 2750 2600 50  0001 C CNN
@@
 	2750 2750 3100 2750
 $Comp
-L power:-VDC #PWR?
+L power:-VDC #PWR07
 U 1 1 5F142F4F
 P 2750 2900
-F 0 "#PWR?" H 2750 2800 50  0001 C CNN
+F 0 "#PWR07" H 2750 2800 50  0001 C CNN
 F 1 "-VDC" H 2750 3175 50  0000 C CNN
 F 2 "" H 2750 2900 50  0001 C CNN
@@
 	2750 2900 3100 2900
 $Comp
-L power:GND #PWR?
+L power:GND #PWR08
 U 1 1 5F145F3E
 P 2900 3250
-F 0 "#PWR?" H 2900 3000 50  0001 C CNN
+F 0 "#PWR08" H 2900 3000 50  0001 C CNN
 F 1 "GND" H 2905 3077 50  0000 C CNN
 F 2 "" H 2900 3250 50  0001 C CNN
